File: Documentation/Circuit/Phone_Finder.sch (KiCad schematic (older format))
At the start: 4 parts

Commit message: Worked on schematic and PCB
Worked on circuit schematic.  Circuits utilized should reflect those in
the BLE112 and AT42 datasheets.  Added initial PCB layout.  Routing
still needs to be done for PCB layout.  Circuit layout should be double
checked before routing.  Refer to an-kd02_103 for more details on touch
interface layout.  Refer to tps62732 datasheet for more details on power
system layout.
Parts:
- added C9: 1uF, ~, symbol C
- gave numbers to parts that had none: 4
Connections:
- net GND: now also C9.2
- net VDD: now also C9.1
- net TOUCH_MODE: now reaches U1.18 (P1_0)
- net TOUCH_OUT: now reaches U1.19 (P0_7)
- no-connect marks 24 -> 22
Changed lines of the file:
@@
 Sheet 1 3
 Title ""
-Date "2 jun 2015"
+Date "4 jun 2015"
 Rev ""
 Comp ""
@@
 $EndDescr
 $Comp
-L BLE112 U?
+L BLE112 U1
 U 1 1 556D11A0
 P 5850 2800
-F 0 "U?" H 5850 2700 50  0000 C CNN
+F 0 "U1" H 5850 2700 50  0000 C CNN
 F 1 "BLE112" H 5850 2900 50  0000 C CNN
 F 2 "MODULE" H 5850 2800 50  0001 C CNN
@@
 F0 "User Input" 50
 F1 "User Input.sch" 50
+F2 "TOUCH_OUT" I R 2200 3300 60
+F3 "TOUCH_MODE" I R 2200 3500 60
 $EndSheet
-Wire Wire Line
-	4600 2200 4600 2300
-Wire Wire Line
-	4600 2300 4800 2300
-Connection ~ 4600 2200
 Text Label 2500 2200 2    60   ~ 0
 DCDC
@@
 	2200 2200 2500 2200
 Wire Wire Line
-	4800 2200 4450 2200
-Wire Wire Line
-	4450 2200 4450 2150
-Wire Wire Line
 	4800 2100 4700 2100
 $Comp
-L GND #PWR?
+L GND #PWR5
 U 1 1 556D35DE
 P 4700 2100
-F 0 "#PWR?" H 4700 2100 30  0001 C CNN
+F 0 "#PWR5" H 4700 2100 30  0001 C CNN
 F 1 "GND" H 4700 2030 30  0001 C CNN
 F 2 "" H 4700 2100 60  0000 C CNN
@@
 	0    1    1    0
 $EndComp
-$Comp
-L VDD #PWR?
-U 1 1 556D35F3
-P 4450 2150
-F 0 "#PWR?" H 4450 2250 30  0001 C CNN
-F 1 "VDD" H 4450 2260 30  0000 C CNN
-F 2 "" H 4450 2150 60  0000 C CNN
-F 3 "" H 4450 2150 60  0000 C CNN
-	1    4450 2150
-	1    0    0    -1
-$EndComp
 Wire Wire Line
 	6000 4000 6000 4550
@@
 	5900 4500 5900 4400
 $Comp
-L VDD #PWR?
+L VDD #PWR7
 U 1 1 556D3668
 P 5900 4400
-F 0 "#PWR?" H 5900 4500 30  0001 C CNN
+F 0 "#PWR7" H 5900 4500 30  0001 C CNN
 F 1 "VDD" H 5900 4510 30  0000 C CNN
 F 2 "" H 5900 4400 60  0000 C CNN
@@
 $EndComp
 Wire Wire Line
-	6100 4000 6100 4200
-$Comp
-L GND #PWR?
-U 1 1 556D3689
-P 6100 4200
-F 0 "#PWR?" H 6100 4200 30  0001 C CNN
-F 1 "GND" H 6100 4130 30  0001 C CNN
-F 2 "" H 6100 4200 60  0000 C CNN
-F 3 "" H 6100 4200 60  0000 C CNN
-	1    6100 4200
-	1    0    0    -1
-$EndComp
-Wire Wire Line
 	4500 2700 4800 2700
 Text Label 4500 2700 0    60   ~ 0
@@
 	3900 2850 3900 2950
 $Comp
-L VDD #PWR?
+L VDD #PWR3
 U 1 1 556D39CC
 P 3900 2850
-F 0 "#PWR?" H 3900 2950 30  0001 C CNN
+F 0 "#PWR3" H 3900 2950 30  0001 C CNN
 F 1 "VDD" H 3900 2960 30  0000 C CNN
 F 2 "" H 3900 2850 60  0000 C CNN
@@
 Connection ~ 3900 2900
 $Comp
-L C C?
+L C C1
 U 1 1 556D39EE
 P 3900 3150
-F 0 "C?" H 3900 3250 40  0000 L CNN
+F 0 "C1" H 3900 3250 40  0000 L CNN
 F 1 "1uF" H 3906 3065 40  0000 L CNN
 F 2 "~" H 3938 3000 30  0000 C CNN
@@
 	3900 3350 3900 3400
 $Comp
-L GND #PWR?
+L GND #PWR4
 U 1 1 556D3A28
 P 3900 3400
-F 0 "#PWR?" H 3900 3400 30  0001 C CNN
+F 0 "#PWR4" H 3900 3400 30  0001 C CNN
 F 1 "GND" H 3900 3330 30  0001 C CNN
 F 2 "" H 3900 3400 60  0000 C CNN
@@
 	4800 3000 4700 3000
 $Comp
-L GND #PWR?
+L GND #PWR6
 U 1 1 556D3A4C
 P 4700 3000
-F 0 "#PWR?" H 4700 3000 30  0001 C CNN
+F 0 "#PWR6" H 4700 3000 30  0001 C CNN
 F 1 "GND" H 4700 2930 30  0001 C CNN
 F 2 "" H 4700 3000 60  0000 C CNN
@@
 Connection ~ 6000 4500
 $Comp
-L C C?
+L C C2
 U 1 1 556D3A7A
 P 6000 4750
-F 0 "C?" H 6000 4850 40  0000 L CNN
+F 0 "C2" H 6000 4850 40  0000 L CNN
 F 1 "1uF" H 6006 4665 40  0000 L CNN
 F 2 "~" H 6038 4600 30  0000 C CNN
@@
 $EndComp
 Wire Wire Line
-	6000 4950 6000 5000
-$Comp
-L GND #PWR?
+	6000 4950 6000 5150
+$Comp
+L GND #PWR8
 U 1 1 556D3AA0
-P 6000 5000
-F 0 "#PWR?" H 6000 5000 30  0001 C CNN
-F 1 "GND" H 6000 4930 30  0001 C CNN
-F 2 "" H 6000 5000 60  0000 C CNN
-F 3 "" H 6000 5000 60  0000 C CNN
-	1    6000 5000
-	1    0    0    -1
-$EndComp
-$Comp
-L GND #PWR?
+P 6000 5150
+F 0 "#PWR8" H 6000 5150 30  0001 C CNN
+F 1 "GND" H 6000 5080 30  0001 C CNN
+F 2 "" H 6000 5150 60  0000 C CNN
+F 3 "" H 6000 5150 60  0000 C CNN
+	1    6000 5150
+	1    0    0    -1
+$EndComp
+$Comp
+L GND #PWR10
 U 1 1 556D3AB8
 P 7100 2700
-F 0 "#PWR?" H 7100 2700 30  0001 C CNN
+F 0 "#PWR10" H 7100 2700 30  0001 C CNN
 F 1 "GND" H 7100 2630 30  0001 C CNN
 F 2 "" H 7100 2700 60  0000 C CNN
@@
 DD
 $Comp
-L CONN_5X2 P?
+L CONN_5X2 P1
 U 1 1 556D3E22
 P 9300 2600
-F 0 "P?" H 9300 2900 60  0000 C CNN
+F 0 "P1" H 9300 2900 60  0000 C CNN
 F 1 "CONN_5X2" V 9300 2600 50  0000 C CNN
 F 2 "" H 9300 2600 60  0000 C CNN
@@
 	8900 2400 8800 2400
 $Comp
-L GND #PWR?
+L GND #PWR11
 U 1 1 556D3E50
 P 8800 2400
-F 0 "#PWR?" H 8800 2400 30  0001 C CNN
+F 0 "#PWR11" H 8800 2400 30  0001 C CNN
 F 1 "GND" H 8800 2330 30  0001 C CNN
 F 2 "" H 8800 2400 60  0000 C CNN
@@
 	9800 2400 9800 2300
 $Comp
-L VDD #PWR?
+L VDD #PWR12
 U 1 1 556D3EB9
 P 9800 2300
-F 0 "#PWR?" H 9800 2400 30  0001 C CNN
+F 0 "#PWR12" H 9800 2400 30  0001 C CNN
 F 1 "VDD" H 9800 2410 30  0000 C CNN
 F 2 "" H 9800 2300 60  0000 C CNN
@@
 NoConn ~ 5600 4000
 NoConn ~ 5700 4000
-NoConn ~ 5900 4000
-NoConn ~ 5800 4000
+Wire Wire Line
+	2200 3300 2500 3300
+Wire Wire Line
+	2200 3500 2500 3500
+Text Label 2500 3300 0    60   ~ 0
+TOUCH_OUT
+Text Label 2500 3500 0    60   ~ 0
+TOUCH_MODE
+Wire Wire Line
+	5800 4000 5800 4150
+Wire Wire Line
+	5800 4150 5100 4150
+Wire Wire Line
+	5900 4000 5900 4250
+Wire Wire Line
+	5900 4250 5100 4250
+Text Label 5100 4250 2    60   ~ 0
+TOUCH_OUT
+Text Label 5100 4150 2    60   ~ 0
+TOUCH_MODE
+Wire Wire Line
+	6100 4000 6100 4250
+$Comp
+L GND #PWR9
+U 1 1 556F7877
+P 6100 4250
+F 0 "#PWR9" H 6100 4250 30  0001 C CNN
+F 1 "GND" H 6100 4180 30  0001 C CNN
+F 2 "" H 6100 4250 60  0000 C CNN
+F 3 "" H 6100 4250 60  0000 C CNN
+	1    6100 4250
+	1    0    0    -1
+$EndComp
+$Comp
+L C C9
+U 1 1 556FEE6E
+P 3650 2550
+F 0 "C9" H 3650 2650 40  0000 L CNN
+F 1 "1uF" H 3656 2465 40  0000 L CNN
+F 2 "~" H 3688 2400 30  0000 C CNN
+F 3 "~" H 3650 2550 60  0000 C CNN
+	1    3650 2550
+	1    0    0    -1
+$EndComp
+Wire Wire Line
+	4800 2200 4700 2200
+Wire Wire Line
+	4700 2200 4700 2300
+Wire Wire Line
+	3650 2300 4800 2300
+Wire Wire Line
+	3650 2250 3650 2350
+Connection ~ 4700 2300
+Connection ~ 3650 2300
+Wire Wire Line
+	3650 2750 3650 2850
+$Comp
+L GND #PWR2
+U 1 1 556FF003
+P 3650 2850
+F 0 "#PWR2" H 3650 2850 30  0001 C CNN
+F 1 "GND" H 3650 2780 30  0001 C CNN
+F 2 "" H 3650 2850 60  0000 C CNN
+F 3 "" H 3650 2850 60  0000 C CNN
+	1    3650 2850
+	1    0    0    -1
+$EndComp
+$Comp
+L VDD #PWR1
+U 1 1 556FF042
+P 3650 2250
+F 0 "#PWR1" H 3650 2350 30  0001 C CNN
+F 1 "VDD" H 3650 2360 30  0000 C CNN
+F 2 "" H 3650 2250 60  0000 C CNN
+F 3 "" H 3650 2250 60  0000 C CNN
+	1    3650 2250
+	1    0    0    -1
+$EndComp
 $EndSCHEMATC

Commit message: Modified input circuitry, remade PCB
Changed input circuit from Atmel's QTouch chipset to a simple momentary
pushbutton, added datasheet for said pushbutton.  Button is dust tight
and waterproof as per spec doc.

Changed passives to use 0603 footprint instead of 0402 to provide easier
reflowing.

Performed initial layout, connectivity, and ground pours.

Still pending are circuit connectivity and feasibility, and PCB
connectivity checks.  Parts might be purchased at this point.  Parts
will then be compared against footprints to ensure fit before sending
gerbers (and order) off to PCB fab.
Connections:
- net STATUS_OUT: now reaches U1.22 (P0_6)
- net TOUCH_MODE: no longer names the net of U1.18 (P1_0)
- net TOUCH_OUT renamed TOUCH_IN
Changed lines of the file:
@@
 Sheet 1 3
 Title ""
-Date "4 jun 2015"
+Date "7 jun 2015"
 Rev ""
 Comp ""
@@
 F0 "User Input" 50
 F1 "User Input.sch" 50
-F2 "TOUCH_OUT" I R 2200 3300 60
-F3 "TOUCH_MODE" I R 2200 3500 60
+F2 "TOUCH_OUT" I R 2200 3200 60
+F3 "STATUS_LED" I R 2200 3500 60
 $EndSheet
 Text Label 2500 2200 2    60   ~ 0
@@
 	4800 2100 4700 2100
 $Comp
-L GND #PWR5
+L GND #PWR01
 U 1 1 556D35DE
 P 4700 2100
-F 0 "#PWR5" H 4700 2100 30  0001 C CNN
+F 0 "#PWR01" H 4700 2100 30  0001 C CNN
 F 1 "GND" H 4700 2030 30  0001 C CNN
 F 2 "" H 4700 2100 60  0000 C CNN
@@
 	5900 4500 5900 4400
 $Comp
-L VDD #PWR7
+L VDD #PWR02
 U 1 1 556D3668
 P 5900 4400
-F 0 "#PWR7" H 5900 4500 30  0001 C CNN
+F 0 "#PWR02" H 5900 4500 30  0001 C CNN
 F 1 "VDD" H 5900 4510 30  0000 C CNN
 F 2 "" H 5900 4400 60  0000 C CNN
@@
 	3900 2850 3900 2950
 $Comp
-L VDD #PWR3
+L VDD #PWR03
 U 1 1 556D39CC
 P 3900 2850
-F 0 "#PWR3" H 3900 2950 30  0001 C CNN
+F 0 "#PWR03" H 3900 2950 30  0001 C CNN
 F 1 "VDD" H 3900 2960 30  0000 C CNN
 F 2 "" H 3900 2850 60  0000 C CNN
@@
 	3900 3350 3900 3400
 $Comp
-L GND #PWR4
+L GND #PWR04
 U 1 1 556D3A28
 P 3900 3400
-F 0 "#PWR4" H 3900 3400 30  0001 C CNN
+F 0 "#PWR04" H 3900 3400 30  0001 C CNN
 F 1 "GND" H 3900 3330 30  0001 C CNN
 F 2 "" H 3900 3400 60  0000 C CNN
@@
 	4800 3000 4700 3000
 $Comp
-L GND #PWR6
+L GND #PWR05
 U 1 1 556D3A4C
 P 4700 3000
-F 0 "#PWR6" H 4700 3000 30  0001 C CNN
+F 0 "#PWR05" H 4700 3000 30  0001 C CNN
 F 1 "GND" H 4700 2930 30  0001 C CNN
 F 2 "" H 4700 3000 60  0000 C CNN
@@
 	6000 4950 6000 5150
 $Comp
-L GND #PWR8
+L GND #PWR06
 U 1 1 556D3AA0
 P 6000 5150
-F 0 "#PWR8" H 6000 5150 30  0001 C CNN
+F 0 "#PWR06" H 6000 5150 30  0001 C CNN
 F 1 "GND" H 6000 5080 30  0001 C CNN
 F 2 "" H 6000 5150 60  0000 C CNN
@@
 $EndComp
 $Comp
-L GND #PWR10
+L GND #PWR07
 U 1 1 556D3AB8
 P 7100 2700
-F 0 "#PWR10" H 7100 2700 30  0001 C CNN
+F 0 "#PWR07" H 7100 2700 30  0001 C CNN
 F 1 "GND" H 7100 2630 30  0001 C CNN
 F 2 "" H 7100 2700 60  0000 C CNN
@@
 	8900 2400 8800 2400
 $Comp
-L GND #PWR11
+L GND #PWR08
 U 1 1 556D3E50
 P 8800 2400
-F 0 "#PWR11" H 8800 2400 30  0001 C CNN
+F 0 "#PWR08" H 8800 2400 30  0001 C CNN
 F 1 "GND" H 8800 2330 30  0001 C CNN
 F 2 "" H 8800 2400 60  0000 C CNN
@@
 	9800 2400 9800 2300
 $Comp
-L VDD #PWR12
+L VDD #PWR09
 U 1 1 556D3EB9
 P 9800 2300
-F 0 "#PWR12" H 9800 2400 30  0001 C CNN
+F 0 "#PWR09" H 9800 2400 30  0001 C CNN
 F 1 "VDD" H 9800 2410 30  0000 C CNN
 F 2 "" H 9800 2300 60  0000 C CNN
@@
 NoConn ~ 6900 3100
 NoConn ~ 6900 3200
-NoConn ~ 6900 3300
-NoConn ~ 6900 3400
-NoConn ~ 6900 3500
 NoConn ~ 4800 3500
 NoConn ~ 4800 3400
@@
 NoConn ~ 5700 4000
 Wire Wire Line
-	2200 3300 2500 3300
-Wire Wire Line
-	2200 3500 2500 3500
-Text Label 2500 3300 0    60   ~ 0
-TOUCH_OUT
-Text Label 2500 3500 0    60   ~ 0
-TOUCH_MODE
-Wire Wire Line
-	5800 4000 5800 4150
-Wire Wire Line
-	5800 4150 5100 4150
+	2200 3200 2500 3200
+Text Label 2500 3200 0    60   ~ 0
+TOUCH_IN
 Wire Wire Line
 	5900 4000 5900 4250
@@
 	5900 4250 5100 4250
 Text Label 5100 4250 2    60   ~ 0
-TOUCH_OUT
-Text Label 5100 4150 2    60   ~ 0
-TOUCH_MODE
+TOUCH_IN
 Wire Wire Line
 	6100 4000 6100 4250
 $Comp
-L GND #PWR9
+L GND #PWR010
 U 1 1 556F7877
 P 6100 4250
-F 0 "#PWR9" H 6100 4250 30  0001 C CNN
+F 0 "#PWR010" H 6100 4250 30  0001 C CNN
 F 1 "GND" H 6100 4180 30  0001 C CNN
 F 2 "" H 6100 4250 60  0000 C CNN
@@
 	3650 2750 3650 2850
 $Comp
-L GND #PWR2
+L GND #PWR011
 U 1 1 556FF003
 P 3650 2850
-F 0 "#PWR2" H 3650 2850 30  0001 C CNN
+F 0 "#PWR011" H 3650 2850 30  0001 C CNN
 F 1 "GND" H 3650 2780 30  0001 C CNN
 F 2 "" H 3650 2850 60  0000 C CNN
@@
 $EndComp
 $Comp
-L VDD #PWR1
+L VDD #PWR012
 U 1 1 556FF042
 P 3650 2250
-F 0 "#PWR1" H 3650 2350 30  0001 C CNN
+F 0 "#PWR012" H 3650 2350 30  0001 C CNN
 F 1 "VDD" H 3650 2360 30  0000 C CNN
 F 2 "" H 3650 2250 60  0000 C CNN
@@
 	1    0    0    -1
 $EndComp
+NoConn ~ 5800 4000
+Wire Wire Line
+	6900 3500 7600 3500
+Text Label 7600 3500 2    60   ~ 0
+STATUS_OUT
+Wire Wire Line
+	2200 3500 2500 3500
+Text Label 2500 3500 0    60   ~ 0
+STATUS_OUT
+NoConn ~ 6900 3300
+NoConn ~ 6900 3400
 $EndSCHEMATC

Commit message: Added BoM, OSHpark estimate
Added BoM, added estimated cost for board fabrication from OSHpark.
Parts:
- C1, C2, C9: footprint ~ -> SM0603_Capa
- P1: footprint (none) -> pinhead-1-2X05SMD/90
- U1: footprint MODULE -> BLE112-A
Changed lines of the file:
@@
 Sheet 1 3
 Title ""
-Date "7 jun 2015"
+Date "11 jun 2015"
 Rev ""
 Comp ""
@@
 F 0 "U1" H 5850 2700 50  0000 C CNN
 F 1 "BLE112" H 5850 2900 50  0000 C CNN
-F 2 "MODULE" H 5850 2800 50  0001 C CNN
+F 2 "BLE112-A" H 5850 2800 50  0001 C CNN
 F 3 "DOCUMENTATION" H 5850 2800 50  0001 C CNN
 	1    5850 2800
@@
 F 0 "C1" H 3900 3250 40  0000 L CNN
 F 1 "1uF" H 3906 3065 40  0000 L CNN
-F 2 "~" H 3938 3000 30  0000 C CNN
+F 2 "SM0603_Capa" H 3938 3000 30  0000 C CNN
 F 3 "~" H 3900 3150 60  0000 C CNN
 	1    3900 3150
@@
 F 0 "C2" H 6000 4850 40  0000 L CNN
 F 1 "1uF" H 6006 4665 40  0000 L CNN
-F 2 "~" H 6038 4600 30  0000 C CNN
+F 2 "SM0603_Capa" H 6038 4600 30  0000 C CNN
 F 3 "~" H 6000 4750 60  0000 C CNN
 	1    6000 4750
@@
 F 0 "P1" H 9300 2900 60  0000 C CNN
 F 1 "CONN_5X2" V 9300 2600 50  0000 C CNN
-F 2 "" H 9300 2600 60  0000 C CNN
+F 2 "pinhead-1-2X05SMD/90" H 9300 2600 60  0000 C CNN
 F 3 "" H 9300 2600 60  0000 C CNN
 	1    9300 2600
@@
 F 0 "C9" H 3650 2650 40  0000 L CNN
 F 1 "1uF" H 3656 2465 40  0000 L CNN
-F 2 "~" H 3688 2400 30  0000 C CNN
+F 2 "SM0603_Capa" H 3688 2400 30  0000 C CNN
 F 3 "~" H 3650 2550 60  0000 C CNN
 	1    3650 2550
