File: Documentation/Circuit/Power Supply.sch (KiCad schematic (older format))
At the start: 6 parts

Commit message: Worked on schematic and PCB
Worked on circuit schematic.  Circuits utilized should reflect those in
the BLE112 and AT42 datasheets.  Added initial PCB layout.  Routing
still needs to be done for PCB layout.  Circuit layout should be double
checked before routing.  Refer to an-kd02_103 for more details on touch
interface layout.  Refer to tps62732 datasheet for more details on power
system layout.
Parts:
- removed BT?: BATTERY, ~, symbol BATTERY
- added BT1: BATTERY, ~, symbol BATTERY
- L1: renamed from L?; value INDUCTOR -> 2.2uH
- gave numbers to parts that had none: 4
Connections:
- net +BATT: now also BT1.1 (+)
- net GND: now also BT1.2 (-)
Other:
- moved on the sheet: C3, C4, C5, L1, U2

Commit message: Added BoM, OSHpark estimate
Added BoM, added estimated cost for board fabrication from OSHpark.
Parts:
- BT1: footprint ~ -> BHX1-2032-SM
- C3: footprint ~ -> SM1206
- C4, C5: footprint ~ -> SM0603_Capa
- L1: footprint ~ -> SM0603
- U2: footprint MODULE -> SON6
Changed lines of the file:
@@
 Sheet 2 3
 Title ""
-Date "7 jun 2015"
+Date "11 jun 2015"
 Rev ""
 Comp ""
@@
 F 0 "U2" H 6750 1700 50  0000 C CNN
 F 1 "TPS62730" H 6750 1900 50  0000 C CNN
-F 2 "MODULE" H 6750 1800 50  0001 C CNN
+F 2 "SON6" H 6750 1800 50  0001 C CNN
 F 3 "DOCUMENTATION" H 6750 1800 50  0001 C CNN
 	1    6750 1800
@@
 F 0 "L1" V 5350 1800 40  0000 C CNN
 F 1 "2.2uH" V 5500 1800 40  0000 C CNN
-F 2 "~" H 5400 1800 60  0000 C CNN
+F 2 "SM0603" H 5400 1800 60  0000 C CNN
 F 3 "~" H 5400 1800 60  0000 C CNN
 	1    5400 1800
@@
 F 0 "C5" H 5000 2500 40  0000 L CNN
 F 1 "2.2uF" H 5006 2315 40  0000 L CNN
-F 2 "~" H 5038 2250 30  0000 C CNN
+F 2 "SM0603_Capa" H 5038 2250 30  0000 C CNN
 F 3 "~" H 5000 2400 60  0000 C CNN
 	1    5000 2400
@@
 F 0 "C3" H 2950 2350 40  0000 L CNN
 F 1 "100uF" H 2956 2165 40  0000 L CNN
-F 2 "~" H 2988 2100 30  0000 C CNN
+F 2 "SM1206" H 2988 2100 30  0000 C CNN
 F 3 "~" H 2950 2250 60  0000 C CNN
 	1    2950 2250
@@
 F 0 "C4" H 4100 2350 40  0000 L CNN
 F 1 "2.2uF" H 4106 2165 40  0000 L CNN
-F 2 "~" H 4138 2100 30  0000 C CNN
+F 2 "SM0603_Capa" H 4138 2100 30  0000 C CNN
 F 3 "~" H 4100 2250 60  0000 C CNN
 	1    4100 2250
@@
 F 0 "BT1" H 3500 2600 50  0000 C CNN
 F 1 "BATTERY" H 3500 2210 50  0000 C CNN
-F 2 "~" H 3500 2400 60  0000 C CNN
+F 2 "BHX1-2032-SM" H 3500 2400 60  0000 C CNN
 F 3 "~" H 3500 2400 60  0000 C CNN
 	1    3500 2400
